Commit message: Cleaning base_optimization package. Created a new package dynamic_obstacle_monitor

File: src/reach_space_modeling/src/generate_pointcloud/model/locobot_wx250s.urdf (robot description, URDF)
Before this commit: robot locobot, 34 links, 33 joints
Links:
- link locobot/ar_tag_link: geometry collision mesh filename=/home/humans/base_seq_opt_multi_dynamic_env_SIM/src/reach_s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 scale=0.001 0.001 0.001; visual mesh filename=/home/humans/base_seq_opt_multi_dynamic_env_SIM/src/reach_s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 scale=0.001 0.001 0.001
- link locobot/arm_base_link: geometry collision mesh filename=/home/humans/base_seq_opt_multi_dynamic_env_SIM/src/reach_s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 scale=0.001 0.001 0.001; visual mesh filename=/home/humans/base_seq_opt_multi_dynamic_env_SIM/src/reach_s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 scale=0.001 0.001 0.001
- link locobot/base_link: geometry collision cylinder length=0.10938 radius=0.178; visual mesh filename=/home/humans/base_seq_opt_multi_dynamic_env_SIM/src/reach_s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
- link locobot/battery_link: geometry collision mesh filename=/home/humans/base_seq_opt_multi_dynamic_env_SIM/src/reach_s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 scale=0.001 0.001 0.001; visual mesh filename=/home/humans/base_seq_opt_multi_dynamic_env_SIM/src/reach_s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 scale=0.001 0.001 0.001
- link locobot/camera_link: geometry collision mesh filename=/home/humans/base_seq_opt_multi_dynamic_env_SIM/src/reach_s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 scale=0.001 0.001 0.001; visual mesh filename=/home/humans/base_seq_opt_multi_dynamic_env_SIM/src/reach_s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 scale=0.001 0.001 0.001
- link locobot/camera_tower_link: geometry collision mesh filename=/home/humans/base_seq_opt_multi_dynamic_env_SIM/src/reach_s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 scale=0.001 0.001 0.001; visual mesh filename=/home/humans/base_seq_opt_multi_dynamic_env_SIM/src/reach_s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 scale=0.001 0.001 0.001
- link locobot/gripper_bar_link: geometry collision mesh filename=/home/humans/base_seq_opt_multi_dynamic_env_SIM/src/reach_s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 scale=0.001 0.001 0.001; visual mesh filename=/home/humans/base_seq_opt_multi_dynamic_env_SIM/src/reach_s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 scale=0.001 0.001 0.001
- link locobot/gripper_link: geometry collision mesh filename=/home/humans/base_seq_opt_multi_dynamic_env_SIM/src/reach_s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 scale=0.001 0.001 0.001; visual mesh filename=/home/humans/base_seq_opt_multi_dynamic_env_SIM/src/reach_s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 scale=0.001 0.001 0.001
- link locobot/gripper_prop_link: geometry collision mesh filename=/home/humans/base_seq_opt_multi_dynamic_env_SIM/src/reach_s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 scale=0.001 0.001 0.001; visual mesh filename=/home/humans/base_seq_opt_multi_dynamic_env_SIM/src/reach_s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 scale=0.001 0.001 0.001
- link locobot/laser_frame_link: geometry collision cylinder length=0.0408 radius=0.03785; visual mesh filename=/home/humans/base_seq_opt_multi_dynamic_env_SIM/src/reach_s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 scale=0.001 0.001 0.001
- link locobot/left_finger_link: geometry collision mesh filename=/home/humans/base_seq_opt_multi_dynamic_env_SIM/src/reach_s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 scale=0.001 0.001 0.001; visual mesh filename=/home/humans/base_seq_opt_multi_dynamic_env_SIM/src/reach_s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 scale=0.001 0.001 0.001
- link locobot/lidar_tower_link: geometry collision mesh filename=/home/humans/base_seq_opt_multi_dynamic_env_SIM/src/reach_s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 scale=0.001 0.001 0.001; visual mesh filename=/home/humans/base_seq_opt_multi_dynamic_env_SIM/src/reach_s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 scale=0.001 0.001 0.001
- link locobot/lower_forearm_link: geometry collision mesh filename=/home/humans/base_seq_opt_multi_dynamic_env_SIM/src/reach_s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 scale=0.001 0.001 0.001; visual mesh filename=/home/humans/base_seq_opt_multi_dynamic_env_SIM/src/reach_s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 scale=0.001 0.001 0.001
- link locobot/pan_link: geometry collision mesh filename=/home/humans/base_seq_opt_multi_dynamic_env_SIM/src/reach_s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 scale=0.001 0.001 0.001; visual mesh filename=/home/humans/base_seq_opt_multi_dynamic_env_SIM/src/reach_s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 scale=0.001 0.001 0.001
- link locobot/plate_link: geometry collision mesh filename=/home/humans/base_seq_opt_multi_dynamic_env_SIM/src/reach_s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 scale=0.001 0.001 0.001; visual mesh filename=/home/humans/base_seq_opt_multi_dynamic_env_SIM/src/reach_s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 scale=0.001 0.001 0.001
- link locobot/right_finger_link: geometry collision mesh filename=/home/humans/base_seq_opt_multi_dynamic_env_SIM/src/reach_s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 scale=0.001 0.001 0.001; visual mesh filename=/home/humans/base_seq_opt_multi_dynamic_env_SIM/src/reach_s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 scale=0.001 0.001 0.001
- link locobot/shoulder_link: geometry collision mesh filename=/home/humans/base_seq_opt_multi_dynamic_env_SIM/src/reach_s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 scale=0.001 0.001 0.001; visual mesh filename=/home/humans/base_seq_opt_multi_dynamic_env_SIM/src/reach_s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 scale=0.001 0.001 0.001
- link locobot/tilt_link: geometry collision mesh filename=/home/humans/base_seq_opt_multi_dynamic_env_SIM/src/reach_s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 scale=0.001 0.001 0.001; visual mesh filename=/home/humans/base_seq_opt_multi_dynamic_env_SIM/src/reach_s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 scale=0.001 0.001 0.001
- link locobot/upper_arm_link: geometry collision mesh filename=/home/humans/base_seq_opt_multi_dynamic_env_SIM/src/reach_s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 scale=0.001 0.001 0.001; visual mesh filename=/home/humans/base_seq_opt_multi_dynamic_env_SIM/src/reach_s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 scale=0.001 0.001 0.001
- link locobot/upper_forearm_link: geometry collision mesh filename=/home/humans/base_seq_opt_multi_dynamic_env_SIM/src/reach_s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 scale=0.001 0.001 0.001; visual mesh filename=/home/humans/base_seq_opt_multi_dynamic_env_SIM/src/reach_s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 scale=0.001 0.001 0.001
- link locobot/wheel_left_link: geometry collision cylinder length=0.0206 radius=0.0352; visual mesh filename=/home/humans/base_seq_opt_multi_dynamic_env_SIM/src/reach_s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
- link locobot/wheel_right_link: geometry collision cylinder length=0.0206 radius=0.0350; visual mesh filename=/home/humans/base_seq_opt_multi_dynamic_env_SIM/src/reach_s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
- link locobot/wrist_link: geometry collision mesh filename=/home/humans/base_seq_opt_multi_dynamic_env_SIM/src/reach_s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 scale=0.001 0.001 0.001; visual mesh filename=/home/humans/base_seq_opt_multi_dynamic_env_SIM/src/reach_s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 scale=0.001 0.001 0.001

File: src/reach_space_modeling/src/generate_pointcloud/model/mobile_wx250s.urdf (robot description, URDF)
Before this commit: robot mobile_wx250s, 15 links, 14 joints
Links:
- link locobot/ar_tag_link: geometry collision mesh filename=/home/humans/base_seq_opt_multi_dynamic_env_SIM/src/reach_s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 scale=0.001 0.001 0.001; visual mesh filename=/home/humans/base_seq_opt_multi_dynamic_env_SIM/src/reach_s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 scale=0.001 0.001 0.001
- link locobot/arm_base_link: geometry collision mesh filename=/home/humans/base_seq_opt_multi_dynamic_env_SIM/src/reach_s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 scale=0.001 0.001 0.001; visual mesh filename=/home/humans/base_seq_opt_multi_dynamic_env_SIM/src/reach_s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 scale=0.001 0.001 0.001
- link locobot/gripper_bar_link: geometry collision mesh filename=/home/humans/base_seq_opt_multi_dynamic_env_SIM/src/reach_s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 scale=0.001 0.001 0.001; visual mesh filename=/home/humans/base_seq_opt_multi_dynamic_env_SIM/src/reach_s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 scale=0.001 0.001 0.001
- link locobot/gripper_link: geometry collision mesh filename=/home/humans/base_seq_opt_multi_dynamic_env_SIM/src/reach_s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 scale=0.001 0.001 0.001; visual mesh filename=/home/humans/base_seq_opt_multi_dynamic_env_SIM/src/reach_s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 scale=0.001 0.001 0.001
- link locobot/gripper_prop_link: geometry collision mesh filename=/home/humans/base_seq_opt_multi_dynamic_env_SIM/src/reach_s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 scale=0.001 0.001 0.001; visual mesh filename=/home/humans/base_seq_opt_multi_dynamic_env_SIM/src/reach_s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 scale=0.001 0.001 0.001
- link locobot/left_finger_link: geometry collision mesh filename=/home/humans/base_seq_opt_multi_dynamic_env_SIM/src/reach_s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 scale=0.001 0.001 0.001; visual mesh filename=/home/humans/base_seq_opt_multi_dynamic_env_SIM/src/reach_s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 scale=0.001 0.001 0.001
- link locobot/lower_forearm_link: geometry collision mesh filename=/home/humans/base_seq_opt_multi_dynamic_env_SIM/src/reach_s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 scale=0.001 0.001 0.001; visual mesh filename=/home/humans/base_seq_opt_multi_dynamic_env_SIM/src/reach_s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 scale=0.001 0.001 0.001
- link locobot/right_finger_link: geometry collision mesh filename=/home/humans/base_seq_opt_multi_dynamic_env_SIM/src/reach_s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 scale=0.001 0.001 0.001; visual mesh filename=/home/humans/base_seq_opt_multi_dynamic_env_SIM/src/reach_s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 scale=0.001 0.001 0.001
- link locobot/shoulder_link: geometry collision mesh filename=/home/humans/base_seq_opt_multi_dynamic_env_SIM/src/reach_s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 scale=0.001 0.001 0.001; visual mesh filename=/home/humans/base_seq_opt_multi_dynamic_env_SIM/src/reach_s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 scale=0.001 0.001 0.001
- link locobot/upper_arm_link: geometry collision mesh filename=/home/humans/base_seq_opt_multi_dynamic_env_SIM/src/reach_s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 scale=0.001 0.001 0.001; visual mesh filename=/home/humans/base_seq_opt_multi_dynamic_env_SIM/src/reach_s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 scale=0.001 0.001 0.001
- link locobot/upper_forearm_link: geometry collision mesh filename=/home/humans/base_seq_opt_multi_dynamic_env_SIM/src/reach_s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 scale=0.001 0.001 0.001; visual mesh filename=/home/humans/base_seq_opt_multi_dynamic_env_SIM/src/reach_s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 scale=0.001 0.001 0.001
- link locobot/wrist_link: geometry collision mesh filename=/home/humans/base_seq_opt_multi_dynamic_env_SIM/src/reach_s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 scale=0.001 0.001 0.001; visual mesh filename=/home/humans/base_seq_opt_multi_dynamic_env_SIM/src/reach_s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 scale=0.001 0.001 0.001
